File: 2613833-Martinez Tagle-microduino/2613833-Martinez Tagle-Microduino.kicad_pcb (KiCad board)
At the start: 2 copper layers, 14 parts, among them J1 USB_A_UCC, J2 Conn_01x10_Socket, U1 ATtiny85-20S

Commit message: Add files via upload
Parts:
- moved J1 11.0 mm to (139.5, 85.7)
- turned D3 to 180 degrees
Routing:
- net GND: track 114.9 -> 3.00 mm
- net Net-(D3-K): track 40.8 -> 0.00 mm
- net +5V: track 32.6 -> 0.00 mm
- net Net-(D5-K): track 19.6 -> 0.00 mm
- net Net-(D1-A): track 16.5 -> 2.00 mm
- net Net-(J2-Pin_4): track 12.7 -> 0.00 mm
- net Net-(J2-Pin_8): track 12.2 -> 0.00 mm
- net Net-(J2-Pin_7): track 11.2 -> 0.00 mm
- net Net-(D3-A): track 9.65 -> 0.00 mm
- net Net-(D2-K): track 19.5 -> 12.1 mm
- net Net-(J2-Pin_6): track 7.29 -> 0.00 mm
- net Net-(J2-Pin_9): track 5.72 -> 0.00 mm
- net Net-(D4-K): track 5.37 -> 0.00 mm
